Commit message: modifiex xacro include command

File: mdr_description/urdf/arm/katana_arm.urdf.xacro (robot description, xacro)
@@ -1,8 +1,8 @@
 <?xml version="1.0"?>
 <robot xmlns:xacro="http://ros.org/wiki/xacro">
-	<include filename="$(find katana_description)/urdf/katana_400_6m180_with_controlbox.urdf.xacro"/>
-	<!-- <include filename="$(find katana_description)/urdf/katana_450_6m90a.urdf.xacro"/> -->
-	<!-- <include filename="$(find katana_description)/urdf/katana_300_6m180.urdf.xacro"/> -->
-	<!-- <include filename="$(find katana_description)/urdf/katana_400_6m180.urdf.xacro"/> -->
+	<xacro:include filename="$(find katana_description)/urdf/katana_400_6m180_with_controlbox.urdf.xacro"/>
+	<!-- <xacro:include filename="$(find katana_description)/urdf/katana_450_6m90a.urdf.xacro"/> -->
+	<!-- <xacro:include filename="$(find katana_description)/urdf/katana_300_6m180.urdf.xacro"/> -->
+	<!-- <xacro:include filename="$(find katana_description)/urdf/katana_400_6m180.urdf.xacro"/> -->
 	<xacro:macro name="katana_arm" params="parent name *origin">
 		<joint name="katana_internal_controlbox_joint" type="fixed">

File: mdr_description/urdf/base/volksbot/base.gazebo.xacro (robot description, xacro)
@@ -33,5 +33,5 @@
 				    <bumperTopicName>${name}_bumper</bumperTopicName>
     			</plugin>
-            </sensor>
+              </sensor>
 			<material>Gazebo/Grey</material>
 		</gazebo>
@@ -50,15 +50,29 @@
 		</gazebo>
 		<gazebo>
-			<plugin name="diffdrive_controller" filename="libdiffdrive_plugin.so">
-				<alwaysOn>true</alwaysOn>
-				<update>100</update>
-				<updateRate>100.0</updateRate>
+                         <plugin name="gazebo_ros_control" filename="libgazebo_ros_control.so">
+                            <robotNamespace>/volksbot</robotNamespace>
+                          </plugin>
+<!--			<plugin name="diffdrive_controller" filename="libdiffdrive_plugin.so"> -->
+			<plugin name="diffdrive_controller" filename="libgazebo_ros_diff_drive.so">
+			  <alwaysOn>true</alwaysOn>
+			  <updateRate>100</updateRate>
+<!--			  <leftJoint>base_link_right_wheel_joint</leftJoint>
+			  <rightJoint>base_link_left_wheel_joint</rightJoint>
+			  <wheelSeparation>0.5380</wheelSeparation>
+			  <wheelDiameter>0.2410</wheelDiameter> -->
+			  <torque>20</torque>
+			  <commandTopic>cmd_vel</commandTopic>
+			  <odometryTopic>odom</odometryTopic>
+			  <odometryFrame>odom</odometryFrame>
+			  <robotBaseFrame>base_footprint</robotBaseFrame>
 				<leftJoint>${name}_link_l_front_wheel_joint</leftJoint>
 				<rightJoint>${name}_link_r_front_wheel_joint</rightJoint>
 				<wheelSeparation>${front_wheel_y * 2}</wheelSeparation>
 				<wheelDiameter>${front_wheel_radius * 2}</wheelDiameter>
+<!--
 				<torque>5</torque>
 				<robotNamespace>/</robotNamespace>
 				<topicName>cmd_vel</topicName>
+				<commandTopic></commandTopic> -->
 			</plugin>
 		</gazebo>

File: mdr_description/urdf/base/volksbot/base.transmission.xacro (robot description, xacro)
@@ -2,10 +2,14 @@
 <robot xmlns:xacro="http://ros.org/wiki/xacro">
 	<!-- Front wheel transmission   -->
-	<xacro:macro name="volksbot_front_wheel_transmission" params="suffix parent reflect">
-		<transmission type="pr2_mechanism_model/SimpleTransmission" name="${parent}_${suffix}_front_wheel_trans">
-			<actuator name="${parent}_${suffix}_front_wheel_motor" />
-			<joint name="${parent}_${suffix}_front_wheel_joint" />
-			<mechanicalReduction>${reflect * 624/35 * 80/18}</mechanicalReduction>
-		</transmission>
+   	<xacro:macro name="volksbot_front_wheel_transmission" params="suffix parent reflect">
+		        <transmission name="${parent}_${suffix}_front_wheel_trans">
+			  <type>transmission_interface/SimpleTransmission</type>
+			  <actuator name="${parent}_${suffix}_front_wheel_motor">
+<!--			    <hardwareInterface>EffortJointInterface</hardwareInterface> -->
+			    <hardwareInterface>VelocityJointInterface</hardwareInterface>
+			    <mechanicalReduction>${reflect * 624/35 * 80/18}</mechanicalReduction>
+			  </actuator>
+			  <joint name="${parent}_${suffix}_front_wheel_joint" />
+			 </transmission>
 	</xacro:macro>
 </robot>

File: mdr_description/urdf/base/volksbot/base.urdf.xacro (robot description, xacro)
@@ -1,8 +1,8 @@
 <?xml version="1.0"?>
 <robot xmlns:xacro="http://ros.org/wiki/xacro">
-	<include filename="$(find mdr_description)/urdf/base/volksbot/base.gazebo.xacro" />
-	<include filename="$(find mdr_description)/urdf/base/volksbot/base.transmission.xacro" />
-	<include filename="$(find mcr_description)/urdf/sensors/sick_lms_200.urdf.xacro"/>
-	<include filename="$(find mcr_description)/urdf/sensors/hokuyo_lx30.urdf.xacro"/>
+	<xacro:include filename="$(find mdr_description)/urdf/base/volksbot/base.gazebo.xacro" />
+	<xacro:include filename="$(find mdr_description)/urdf/base/volksbot/base.transmission.xacro" />
+	<xacro:include filename="$(find mcr_description)/urdf/sensors/sick_lms_200.urdf.xacro"/>
+	<xacro:include filename="$(find mcr_description)/urdf/sensors/hokuyo_lx30.urdf.xacro"/>
 	<!-- base -->
 	<property name="base_width" value="0.5" />
@@ -142,5 +142,5 @@
 			</visual>
 			<collision>
-				<origin xyz="0 0 0" rpy="0 0 0" />
+				<origin xyz="0 0 0.1" rpy="0 0 0" />
 				<geometry>
 					<box size="0.001 0.001 0.001" />

File: mdr_description/urdf/head/volksbot/head.urdf.xacro (robot description, xacro)
@@ -2,5 +2,8 @@
 <robot xmlns:xacro="http://ros.org/wiki/xacro">
 	<!-- kinect -->
-	<include filename="$(find mcr_description)/urdf/sensors/kinect.urdf.xacro"/>
+<!--
+	<xacro:include filename="$(find mdr_description)/urdf/head/volksbot/head.transmission.xacro" />
+-->
+        <xacro:include filename="$(find mcr_description)/urdf/sensors/kinect_camera.urdf.xacro"/>
 	<xacro:macro name="volksbot_head" params="parent name *origin">
 		<link name="${name}_camera_link" />
@@ -11,7 +14,10 @@
 		</joint>
 		<!-- kinect -->
-		<xacro:kinect name="openni" ros_topic="/cam3d/depth/points1" parent="${name}_camera_link">
+		<xacro:kinect_camera name="openni" parent="${name}_camera_link">
 			<origin xyz="0 0 0.01" rpy="0 0 ${M_PI}" />
-		</xacro:kinect>
+		</xacro:kinect_camera>
+<!--
+		<xacro:volksbot_ptu_transmission name="${name}"/>
+-->
 	</xacro:macro>
 </robot>

File: mdr_description/urdf/torso/volksbot/torso.urdf.xacro (robot description, xacro)
@@ -1,5 +1,5 @@
 <?xml version="1.0"?>
 <robot xmlns:xacro="http://ros.org/wiki/xacro">
-	<include filename="$(find mdr_description)/urdf/torso/volksbot/torso.gazebo.xacro" />
+	<xacro:include filename="$(find mdr_description)/urdf/torso/volksbot/torso.gazebo.xacro" />
 	<xacro:macro name="volksbot_torso" params="parent name *origin">
 		<link name="${name}_lower_link">

File: mdr_hardware_config/volksbot/urdf/volksbot.urdf.xacro (robot description, xacro)
@@ -2,19 +2,19 @@
 <robot xmlns:xacro="http://ros.org/wiki/xacro" name="volksbot">
 	<!-- common definitions -->
-	<include filename="$(find mdr_description)/urdf/common.xacro" />
+	<xacro:include filename="$(find mcr_description)/urdf/common.xacro" />
 	<!-- calibration -->
-	<include filename="$(find mdr_calibration_data)/$(env ROBOT)/calibration/calibration.urdf.xacro" />
+	<xacro:include filename="$(find mdr_calibration_data)/$(env ROBOT)/calibration/calibration.urdf.xacro" />
 	<!-- materials for visualization -->
-	<include filename="$(find mdr_description)/urdf/materials.urdf.xacro" />
+	<xacro:include filename="$(find mcr_description)/urdf/materials.urdf.xacro" />
 	<!-- base -->
-	<include filename="$(find mdr_description)/urdf/base/volksbot/base.urdf.xacro"/>
+	<xacro:include filename="$(find mdr_description)/urdf/base/volksbot/base.urdf.xacro"/>
 	<!-- torso -->
-	<include filename="$(find mdr_description)/urdf/torso/volksbot/torso.urdf.xacro"/>
+	<xacro:include filename="$(find mdr_description)/urdf/torso/volksbot/torso.urdf.xacro"/>
 	<!-- ptu -->
-	<include filename="$(find mcr_description)/urdf/ptu/ptu46.urdf.xacro"/>
+	<xacro:include filename="$(find mcr_description)/urdf/ptu/ptu46.urdf.xacro"/>
 	<!-- head -->
-	<include filename="$(find mdr_description)/urdf/head/volksbot/head.urdf.xacro"/>
+	<xacro:include filename="$(find mdr_description)/urdf/head/volksbot/head.urdf.xacro"/>
 	<!-- arm -->
-	<include filename="$(find mdr_description)/urdf/arm/katana_arm.urdf.xacro"/>
+	<xacro:include filename="$(find mdr_description)/urdf/arm/katana_arm.urdf.xacro"/>
 	<xacro:volksbot_base name="base"/>
 	<xacro:volksbot_torso name="torso" parent="base_upper_case_link">
