Commit message: update cob3-1 urdf in moveit config

File: mdr_moveit_cob/config/cob3_1.urdf (robot description, URDF)
Before this commit: robot cob3-1, 56 links, 55 joints
Links:
- added link lookat_base_link
- added link lookat_focus_frame
- added link lookat_x_link
- added link lookat_y_link
- added link lookat_z_link
- link base_link: geometry collision mesh filename=package://cob_description/meshes/cob3_base/base_collision.s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; visual mesh filename=package://cob_description/meshes/cob3_base/base.stl
- link bl_caster_rotation_link: geometry collision box size=0.001 0.001 0.001; visual mesh filename=package://cob_description/meshes/cob3_base/caster.stl
- link br_caster_rotation_link: geometry collision box size=0.001 0.001 0.001; visual mesh filename=package://cob_description/meshes/cob3_base/caster.stl
- link fl_caster_rotation_link: geometry collision box size=0.001 0.001 0.001; visual mesh filename=package://cob_description/meshes/cob3_base/caster.stl
- link fr_caster_rotation_link: geometry collision box size=0.001 0.001 0.001; visual mesh filename=package://cob_description/meshes/cob3_base/caster.stl
- link head_cam3d_link: geometry collision box size=0.06 0.02 0.02; visual box size=0.06 0.02 0.02
- link head_color_camera_l_link: geometry collision cylinder length=0.03 radius=0.01; visual cylinder length=0.03 radius=0.01
- link head_color_camera_r_link: geometry collision cylinder length=0.03 radius=0.01; visual cylinder length=0.03 radius=0.01
- link head_cover_link: geometry collision mesh filename=package://cob_description/meshes/cob3_torso/head_cover_coll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; visual mesh filename=package://cob_description/meshes/cob3_torso/head_cover.stl
- link torso_lower_neck_tilt_link: geometry collision mesh filename=package://cob_description/meshes/cob3_torso/lower_neck_coll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; visual mesh filename=package://cob_description/meshes/cob3_torso/lower_neck.stl
- link torso_upper_neck_tilt_link: geometry collision mesh filename=package://cob_description/meshes/cob3_torso/upper_neck.stl; visual mesh filename=package://cob_description/meshes/cob3_torso/upper_neck.stl
- link tray_link: geometry collision mesh filename=package://cob_description/meshes/cob3_tray/tray_collision.s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; visual mesh filename=package://cob_description/meshes/cob3_tray/tray.stl
Joints:
- added joint lookat_base_joint: type fixed, parent torso_upper_neck_tilt_link, child lookat_base_link, origin xyz=0.0 -0.154 0.0 rpy=3.1415926 3.1415926 3.14159265359
- added joint lookat_lin_joint: type prismatic, parent lookat_base_link, child lookat_x_link, origin xyz=0 0 0 rpy=0 0 0, axis -1 0 0, limit lower=-5.0 upper=5.0 effort=100 velocity=1
- added joint lookat_x_joint: type revolute, parent lookat_x_link, child lookat_y_link, origin xyz=0 0 0 rpy=0 0 0, axis 1 0 0, limit lower=-3.14159265359 upper=3.14159265359 effort=100 velocity=1
- added joint lookat_y_joint: type revolute, parent lookat_y_link, child lookat_z_link, origin xyz=0 0 0 rpy=0 0 0, axis 0 1 0, limit lower=-3.14159265359 upper=3.14159265359 effort=100 velocity=1
- added joint lookat_z_joint: type revolute, parent lookat_z_link, child lookat_focus_frame, origin xyz=0 0 0 rpy=0 0 0, axis 0 0 1, limit lower=-3.14159265359 upper=3.14159265359 effort=100 velocity=1
- joint head_cam3d_joint: origin xyz=-0.06 0.055 0.0 rpy=1.57079632679 -1.57079632679 0.0 -> xyz=-0.09 0.095 0.02 rpy=1.57079632679 -1.57079632679 0.0
- joint torso_lower_neck_pan_joint: limit lower=-1.0 upper=1.0 effort=24 velocity=0.5 -> lower=-0.1 upper=0.1 effort=200 velocity=0.5
- joint torso_lower_neck_tilt_joint: limit lower=-0.4 upper=0.4 effort=46 velocity=0.5 -> lower=-0.26 upper=0.25 effort=200 velocity=0.5
- joint torso_upper_neck_pan_joint: limit lower=-1.0 upper=1.0 effort=4 velocity=0.5 -> lower=-0.2 upper=0.2 effort=200 velocity=0.5
- joint torso_upper_neck_tilt_joint: limit lower=-0.4 upper=0.4 effort=24 velocity=0.5 -> lower=-0.21 upper=0.3 effort=200 velocity=0.5
